Commit message: Created core URDF

File: description/robot.urdf.xacro (robot description, xacro)
@@ -2,4 +2,9 @@
 <robot xmlns:xacro="http://www.ros.org/wiki/xacro"  name="robot">
    <xacro:include filename="robot_core.xacro" />
-    <xacro:include filename="gazebo_control.xacro"/>
+   <!--<xacro:include filename="gazebo_control.xacro"/> -->
+   <xacro:include filename="ros2_control.xacro"/>
+   <xacro:include filename="lidar.xacro"/>
+   <xacro:include filename="camera.xacro"/>
+    <xacro:include filename="face.xacro" />
+   <!--<xacro:include filename="depth_camera.xacro"/> -->
 </robot>

File: description/robot_core.xacro (robot description, xacro)
@@ -2,4 +2,18 @@
 <robot xmlns:xacro="http://www.ros.org/wiki/xacro" >
   <xacro:include filename="inertial_macros.xacro"/>
+   <xacro:property name="chassis_length" value="0.335"/>
+    <xacro:property name="chassis_width" value="0.265"/>
+    <xacro:property name="chassis_height" value="0.138"/>
+    <xacro:property name="chassis_mass" value="1.0"/>
+    <xacro:property name="wheel_radius" value="0.034"/>
+    <xacro:property name="wheel_thickness" value="0.026"/>
+    <xacro:property name="wheel_mass" value="0.05"/>
+    <xacro:property name="wheel_offset_x" value="0.226"/>
+    <xacro:property name="wheel_offset_y" value="0.166"/>
+    <xacro:property name="wheel_offset_z" value="0.01"/>
+    <xacro:property name="caster_wheel_radius" value="0.01"/>
+    <xacro:property name="caster_wheel_mass" value="0.01"/>
+    <xacro:property name="caster_wheel_offset_x" value="0.075"/>
+    <xacro:property name="caster_wheel_offset_z" value="${wheel_offset_z - wheel_radius + caster_wheel_radius}"/>
   <material name="white">
     <color rgba="1 1 1 1"/>
@@ -14,4 +28,7 @@
     <color rgba="0 0 0 1"/>
   </material>
+  <material name="red">
+    <color rgba="1 0 0 1"/>
+  </material>
   <!--BASE LINK-->
   <link name="base_link"></link>
@@ -20,27 +37,27 @@
     <parent link="base_link"/>
     <child link="chassis"/>
-    <origin xyz="-0.1 0 0"/>
+    <origin xyz="${-wheel_offset_x} 0 ${-wheel_offset_z}"/>
   </joint>
   <link name="chassis">
     <visual>
-      <origin xyz="0.15 0 0.075"/>
+       <origin xyz="${chassis_length/2} 0 ${chassis_height/2}"/>
       <geometry>
-        <box size="0.3 0.3 0.15"/>
+        <box size="${chassis_length} ${chassis_width} ${chassis_height}"/>
       </geometry>
-      <material name="white"/>
+      <material name="orange"/>
     </visual>
     <collision>
-      <origin xyz="0.15 0 0.075"/>
+      <origin xyz="${chassis_length/2} 0 ${chassis_height/2}"/>
       <geometry>
-        <box size="0.3 0.3 0.15"/>
+        <box size="${chassis_length} ${chassis_width} ${chassis_height}"/>
       </geometry>
       <material name="white"/>
     </collision>
-    <xacro:inertial_box mass="0.5" x="0.3" y="0.3" z="0.15">
-      <origin xyz="0.15 0 0.075" rpy="0 0 0"/>
+    <xacro:inertial_box mass="0.5" x="${chassis_length}" y="${chassis_width}" z="${chassis_height}">
+          <origin xyz="${chassis_length/2} 0 ${chassis_height/2}" rpy="0 0 0"/>
     </xacro:inertial_box>
   </link>
    <gazebo reference="chassis">
-        <material>Gazebo/White</material>
+        <material>Gazebo/Orange</material>
   </gazebo>
   <!--LEFT WHEEL-->
@@ -48,5 +65,5 @@
     <parent link="base_link"/>
     <child link="left_wheel"/>
-    <origin xyz="0 0.175 0" rpy="-${pi/2} 0 0"/>
+    <origin xyz="0 ${wheel_offset_y} 0" rpy="-${pi/2} 0 0" />
     <axis xyz="0 0 1"/>
   </joint>
@@ -54,5 +71,5 @@
     <visual>
       <geometry>
-        <cylinder radius="0.05" length="0.04"/>
+        <cylinder radius="${wheel_radius}" length="${wheel_thickness}"/>
       </geometry>
       <material name="blue"/>
@@ -60,9 +77,9 @@
     <collision>
       <geometry>
-        <cylinder radius="0.05" length="0.04"/>
+        <sphere radius="${wheel_radius}"/>
       </geometry>
       <material name="blue"/>
     </collision>
-    <xacro:inertial_cylinder mass="0.1" length="0.04" radius="0.05">
+    <xacro:inertial_cylinder mass="${wheel_mass}" length="${wheel_thickness}" radius="${wheel_radius}">
       <origin xyz="0 0 0" rpy="0 0 0"/>
     </xacro:inertial_cylinder>
@@ -75,5 +92,5 @@
     <parent link="base_link"/>
     <child link="right_wheel"/>
-    <origin xyz="0 -0.175 0" rpy="${pi/2} 0 0"/>
+    <origin xyz="0 ${-wheel_offset_y} 0" rpy="${pi/2} 0 0" />
     <axis xyz="0 0 -1"/>
   </joint>
@@ -81,5 +98,5 @@
     <visual>
       <geometry>
-        <cylinder radius="0.05" length="0.04"/>
+        <cylinder radius="${wheel_radius}" length="${wheel_thickness}"/>
       </geometry>
       <material name="blue"/>
@@ -87,9 +104,9 @@
     <collision>
       <geometry>
-        <cylinder radius="0.05" length="0.04"/>
+        <sphere radius="${wheel_radius}"/>
       </geometry>
       <material name="blue"/>
     </collision>
-    <xacro:inertial_cylinder mass="0.1" length="0.04" radius="0.05">
+    <xacro:inertial_cylinder mass="${wheel_mass}" length="${wheel_thickness}" radius="${wheel_radius}">
       <origin xyz="0 0 0" rpy="0 0 0"/>
     </xacro:inertial_cylinder>
@@ -102,25 +119,25 @@
     <parent link="chassis"/>
     <child link="caster_wheel"/>
-    <origin xyz="0.24 0 0"/>
+    <origin xyz="${caster_wheel_offset_x} 0 ${caster_wheel_offset_z}"/>
   </joint>
   <link name="caster_wheel">
     <visual>
       <geometry>
-        <sphere radius="0.05"/>
+        <sphere radius="${caster_wheel_radius}"/>
       </geometry>
-      <material name="black"/>
+      <material name="white"/>
     </visual>
     <collision>
         <geometry>
-            <sphere radius="0.05"/>
+             <sphere radius="${caster_wheel_radius}"/>
         </geometry>
         <material name="black"/>
     </collision>
-    <xacro:inertial_sphere mass="0.1" radius="0.05">
+    <xacro:inertial_sphere mass="${caster_wheel_mass}" radius="${caster_wheel_radius}">
         <origin xyz="0 0 0" rpy="0 0 0"/>
     </xacro:inertial_sphere>
 </link>
  <gazebo reference="caster_wheel">
-        <material>Gazebo/Black</material>
+        <material>Gazebo/White</material>
         <mu1 value="0.001"/>
         <mu2 value="0.001"/>
